File: eecd_project/eecd_project.kicad_sch (KiCad schematic)
At the start: 0 parts

Commit message: before relays
Parts:
- added C1, C2: 22p, symbol Device:C_Small
- added C10, C5, C7: 100nF, symbol Device:C_Small
- added C3, C9: 1uF, symbol Device:C_Small
- added C4: 4.7uF, symbol Device:C_Small
- added C6: 4.7u, symbol Device:C_Small
- added C8: 10uF, symbol Device:C_Small
- added IC1: LMR54406FDBVR, SOT95P280X145-6N, symbol LMR54406FDBVR:LMR54406FDBVR
- added J1: Conn_02x07_Counter_Clockwise, symbol Connector_Generic:Conn_02x07_Counter_Clockwise
- added L1: 12uH, symbol Device:L
- added R1, R2, R3, R4: 10k, symbol Device:R
- added R5: 69k8, symbol Device:R
- added R6: 22k1, symbol Device:R
- added SW1: SW_Push, symbol Switch:SW_Push
- added U1: ATmega32A-A, Package_QFP:TQFP-44_10x10mm_P0.8mm, symbol MCU_Microchip_ATmega:ATmega32A-A
- added U2: ESP8266-12E_ESP-12E, ESP8266-12E_ESP-12E:XCVR_ESP8266-12E_ESP-12E, symbol ESP8266-12E_ESP-12E:ESP8266-12E_ESP-12E
- added Y1: 8MHz, symbol Device:Crystal
Connections:
- new net: C7.1, IC1.6 (SW), L1.1
- new net: C7.2, IC1.1 (CB)
- new net: C10.2, C8.2, C9.2, IC1.2 (GND), R6.2
- new net: C3.1, C4.1, R3.1, U2.8 (VCC)
- new net: J1.14 (Pin_14), R1.2
- new net: C2.1, U1.8 (XTAL1), Y1.1
- new net: C1.1, U1.7 (XTAL2), Y1.2
- new net: R3.2, U2.3 (EN)
- new net: R4.1, U2.16 (IO15)
- new net: IC1.3 (FB), R5.2, R6.1
- new net +24V: C10.1, C9.1, IC1.4 (EN), IC1.5 (VIN)
- new net +3.3V: C8.1, J1.1 (Pin_1), L1.2, R5.1
- new net ???: U2.17 (IO2), U2.18 (IO0)
- new net AM: J1.4 (Pin_4), U1.42 (PB2)
- new net CD: J1.12 (Pin_12), U1.41 (PB1)
- new net DR: J1.11 (Pin_11), U1.43 (PB3)
- new net GND: C1.2, C2.2, C3.2, C4.2, C5.2, C6.2, J1.7 (Pin_7), J1.8 (Pin_8), R1.1, R2.2, R4.2, U1.18 (GND), U1.28 (GND), U1.39 (GND), U1.6 (GND), U2.15 (GND)
- new net IN1: U1.19 (PC0)
- new net IN2: U1.20 (PC1)
- new net IN3: U1.21 (PC2)
- new net IN4: U1.22 (PC3)
- new net MISO: J1.5 (Pin_5), U1.2 (PB6)
- new net MOSI: J1.10 (Pin_10), U1.1 (PB5)
- new net OUT1: U1.23 (PC4)
- new net OUT2: U1.24 (PC5)
- new net OUT3: U1.25 (PC6)
- new net OUT4: U1.26 (PC7)
- new net RESET: R2.1, SW1.1, U1.4 (~{RESET}), U2.1 (RESET)
- new net RHR?: J1.13 (Pin_13)
- new net RXD: U1.9 (PD0), U2.22 (TXD)
- new net SCK: J1.6 (Pin_6), U1.3 (PB7)
- new net TXD: U1.10 (PD1), U2.21 (RXD)
- new net UCK?: J1.3 (Pin_3)
- new net VDD: C5.1, C6.1, SW1.2, U1.17 (VCC), U1.27 (AVCC), U1.38 (VCC), U1.5 (VCC)
- new net ~{SS}: J1.9 (Pin_9), U1.44 (PB4)
- no-connect marks 0 -> 29
Other:
- removed sheet gate controller
- removed sheet key fob
- added sheet inputs_outputs (io.kicad_sch)
- note added: "???"
- note added: "TODO: Qty means series or parallel?"
- note added: "bypass capacitors for modules?"
- note added: "nRF905 module connector"

Commit message: v1
Parts:
- added C11, C12: 1uF, symbol Device:C_Small
- added C13: 10uF, symbol Device:C_Small
- C1, C2: value 22p -> 22pF
Connections:
- net +3.3V is gone; now on net VDD: C8.1, J1.1 (Pin_1), L1.2, R5.1
- net +24V: now also C11.1, C12.1
- net VDD: now also C3.1, C4.1, J1.2 (Pin_2), R3.1, U2.8 (VCC), C13.1
- net at C10.2, C8.2, C9.2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: now also C11.2, C12.2, C13.2
- net ??? renamed PULL_UP2?
- net PULL_UP2?: no longer U2.17 (IO2)
- new net PULL_UP?: U2.17 (IO2)
Other:
- sheet inputs_outputs ports: added IN1, IN2, IN3, IN4, OUT1, OUT2, OUT3, OUT4; removed none
- note added: "pull up R?"
- note removed: "???"
- note removed: "TODO: Qty means series or parallel?"
- note removed: "bypass capacitors for modules?"
- moved on the sheet: C10, C7, C8, C9, IC1, L1, R2, R5, R6, SW1

Commit message: v2
Parts:
- added R27, R28, R29: 10K, symbol Device:R
- R1, R3, R4: value 10k -> 10K
- R2: value 10k -> ESP_RESET
- R5: value 69k8 -> 69K8
- R6: value 22k1 -> 22K1
Connections:
- net GND: now also R1.2; no longer R1.1
- net RESET: no longer U2.1 (RESET)
- net VDD: now also R27.1, R28.1, R29.2; no longer J1.2 (Pin_2)
- net at J1.14 (Pin_14): now also R1.1; no longer R1.2
- net ESP_RESET: now reaches U1.11 (PD2)
- net ESP_RESET: now also U2.1 (RESET)
- net TRX_CE: now reaches U1.40 (PB0)
- net TRX_CE: now also J1.2 (Pin_2)
- net PULL_UP2?: no longer names the net of U2.18 (IO0)
- net PULL_UP2?: now also R27.2
- net PULL_UP?: no longer names the net of U2.17 (IO2)
- net PULL_UP?: now also R28.2
- net RHR?: no longer names the net of J1.13 (Pin_13)
- net RHR?: now also R29.1
- net UCK?: no longer names the net of J1.3 (Pin_3)
- no-connect marks 29 -> 28
Other:
- note added: "ESP12-E"
- note added: "Inputs and outputs"
- note added: "Microcontroller - ATMega32-A"
- note added: "Microcontroller reset switch"
- note added: "Power supply"
- note removed: "pull up R?"
- moved on the sheet: C1, C10, C11, C12, C13, C2, C3, C4, C5, C6, C7, C8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

Commit message: v3
Parts:
- added D5, D6: LED, symbol Device:LED
- added F1: 600mA, symbol Device:Fuse
- added J11: Conn_01x06, symbol Connector_Generic:Conn_01x06
- added J7: Barrel_Jack, symbol Connector:Barrel_Jack
- added R30: 10K, symbol Device:R
- added R31: 47R, symbol Device:R
- added R32: 100R, symbol Device:R
- C10: QTY Qty=2 -> (none); V (none) -> 35V
- C11, C12, C9: V (none) -> 35V
- R2: value ESP_RESET -> 10K
Connections:
- net +24V: now also F1.1, J7.1; no longer C10.1, C11.1, C12.1, C9.1, IC1.4 (EN), IC1.5 (VIN)
- net GND: now also C10.2, C11.2, C12.2, C13.2, C8.2, C9.2, IC1.2 (GND), R6.2, D5.1 (K), D6.1 (K), J11.6 (Pin_6), J7.2
- net MISO: now also J11.2 (Pin_2)
- net MOSI: now also J11.3 (Pin_3)
- net RESET: now also J11.1 (Pin_1)
- net SCK: now also J11.4 (Pin_4)
- net VDD: now also J11.5 (Pin_5), R30.2
- net ~{SS}: now also R30.1
- net STATUS_OK: now reaches U1.12 (PD3)
- net STATUS_OK: now also R31.1
- net STATUS_ERROR: now reaches U1.13 (PD4)
- net STATUS_ERROR: now also R32.1
- net ESP_RESET renamed ~{ESP_RESET}
- new net: D5.2 (A), R31.2
- new net: C10.1, C11.1, C12.1, C9.1, F1.2, IC1.4 (EN), IC1.5 (VIN)
- new net: D6.2 (A), R32.2
- no-connect marks 28 -> 26
Other:
- note added: "Programmer connector"
- moved on the sheet: R1, R29

Commit message: ?
Changed lines of the file:
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@@
+    )
+  )
+  (symbol (lib_id "Device:R") (at 347.98 72.39 0) (unit 1)
+    (in_bom yes) (on_board yes) (dnp no) (fields_autoplaced)
+    (property "Reference" "R1" (at 350.52 71.12 0)
+      (effects (font (size 1.27 1.27)) (justify left))
+    )
+    (property "Value" "10K" (at 350.52 73.66 0)
+      (effects (font (size 1.27 1.27)) (justify left))
+    )
+    (property "Footprint" "" (at 346.202 72.39 90)
+      (effects (font (size 1.27 1.27)) hide)
+    )
+    (property "Datasheet" "~" (at 347.98 72.39 0)
+      (effects (font (size 1.27 1.27)) hide)
+    )
+    (pin "1")
+    (pin "2")
+    (instances
+      (project "eecd_project"
+        (path "/ab78a217-a529-4c6b-b5ff-15aec0144b8e"
+          (reference "R1") (unit 1)
+        )
+      )
     )
   )
@@
         )
       )
-    )
-  )
-  (symbol (lib_id "Device:R") (at 347.98 72.39 0) (unit 1)
-    (in_bom yes) (on_board yes) (dnp no)
-    (property "Reference" "R1" (at 341.63 72.39 90)
-      (effects (font (size 1.27 1.27)))
-    )
-    (property "Value" "10K" (at 344.17 72.39 90)
-      (effects (font (size 1.27 1.27)))
-    )
-    (property "Footprint" "" (at 346.202 72.39 90)
-      (effects (font (size 1.27 1.27)) hide)
-    )
-    (property "Datasheet" "~" (at 347.98 72.39 0)
-      (effects (font (size 1.27 1.27)) hide)
-    )
-    (pin "1")
-    (pin "2")
-    (instances
-      (project "eecd_project"
-        (path "/ab78a217-a529-4c6b-b5ff-15aec0144b8e"
-          (reference "R1") (unit 1)
-        )
-      )

Commit message: ?
Parts:
- removed J1: Conn_02x07_Counter_Clockwise, symbol Connector_Generic:Conn_02x07_Counter_Clockwise
- added J1: Conn_02x07_Odd_Even, Connector_PinSocket_2.54mm:PinSocket_2x07_P2.54mm_Vertical, symbol Connector_Generic:Conn_02x07_Odd_Even
- C1, C10, C11, C12, C13, C2, C3, C4, C5, C7, C8, C9: footprint (none) -> Capacitor_SMD:C_0603_1608Metric_Pad1.08x0.95mm_HandSolder
- C6: value 4.7u -> 4.7uF; footprint (none) -> Capacitor_SMD:C_0603_1608Metric_Pad1.08x0.95mm_HandSolder
- D5: footprint (none) -> LED_SMD:LED_0603_1608Metric_Pad1.05x0.95mm_HandSolder; Field5 V_{f} = 2.4V -> V_{f} = 2.1V
- D6: footprint (none) -> LED_SMD:LED_0603_1608Metric_Pad1.05x0.95mm_HandSolder
- F1: footprint (none) -> Fuse:Fuseholder_Clip-5x20mm_Littelfuse_445-030_Inline_P20.50x5.20mm_D1.30mm_Horizontal
- IC1: footprint SOT95P280X145-6N -> LIB_LMR54406FDBVR:SOT95P280X145-6N
- J11: footprint (none) -> Connector_Molex:Molex_PicoBlade_53047-0610_1x06_P1.25mm_Vertical
- J7: footprint (none) -> Connector_BarrelJack:BarrelJack_CUI_PJ-063AH_Horizontal
- L1: footprint (none) -> Inductor_SMD:L_Bourns-SRN4018
- R1, R2, R27, R28, R29, R3, R30, R32, R4, R5, R6: footprint (none) -> Resistor_SMD:R_0603_1608Metric_Pad0.98x0.95mm_HandSolder
- R31: value 47R -> 100R; footprint (none) -> Resistor_SMD:R_0603_1608Metric_Pad0.98x0.95mm_HandSolder
- SW1: footprint (none) -> Button_Switch_THT:SW_Tactile_SPST_Angled_PTS645Vx83-2LFS
- U2: footprint ESP8266-12E_ESP-12E:XCVR_ESP8266-12E_ESP-12E -> LIB_ESP8266-12E_ESP-12E:XCVR_ESP8266-12E_ESP-12E
- Y1: footprint (none) -> LIB_CRYSTAL:XTAL_ABLS2_ABR
Connections:
- net AM: now also U1.41 (PB1), J1.8 (Pin_8); no longer U1.42 (PB2)
- net CD: now also U1.42 (PB2), J1.5 (Pin_5); no longer U1.41 (PB1)
- net DR: now also U1.40 (PB0), J1.7 (Pin_7); no longer U1.43 (PB3)
- net GND: now also J1.13 (Pin_13), J1.14 (Pin_14)
- net IN1: now also U1.23 (PC4); no longer U1.19 (PC0)
- net IN2: now also U1.24 (PC5); no longer U1.20 (PC1)
- net IN3: now also U1.25 (PC6); no longer U1.21 (PC2)
- net IN4: now also U1.26 (PC7); no longer U1.22 (PC3)
- net MISO: now also J1.10 (Pin_10)
- net MOSI: now also J1.9 (Pin_9)
- net OUT1: now also U1.22 (PC3); no longer U1.23 (PC4)
- net OUT2: now also U1.21 (PC2); no longer U1.24 (PC5)
- net OUT3: now also U1.20 (PC1); no longer U1.25 (PC6)
- net OUT4: now also U1.19 (PC0); no longer U1.26 (PC7)
- net SCK: now also J1.12 (Pin_12)
- net TRX_CE: now also U1.43 (PB3), J1.4 (Pin_4); no longer U1.40 (PB0)
- net VDD: now also J1.2 (Pin_2)
- net ~{SS}: now also J1.11 (Pin_11)
- net at R29.1: now also J1.3 (Pin_3)
- net at R1.1: now also J1.1 (Pin_1)
Other:
- company: (none) -> Mateusz Pietrzak, Ruman Mondal, Bassey Bassey
- title: (none) -> Gate controller
