File: eecd_project/io.kicad_sch (KiCad schematic)
At the start: 43 parts, among them J2 Screw_Terminal_01x04, J3 Screw_Terminal_01x03, J4 Screw_Terminal_01x03, J5 Screw_Terminal_01x03, J6 Screw_Terminal_01x03, K1 PE014024, K2 PE014024, K3 PE014024, K4 PE014024, Q1 MMBT3906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

Commit message: v2
Parts:
- removed Q1, Q2, Q3, Q4: MMBT3906, Package_TO_SOT_SMD:SOT-23, symbol Transistor_BJT:MMBT3906
- R10, R14, R8: value 10k -> 10K
- R11, R12, R15, R17, R18, R19, R20, R21, R22, R23, R24, R25, R26, R7, R9: value 470 -> 470R
- R13: value 10k -> 470R
- R16: value 470 -> 10K
Connections:
- net GND: now also R16.2; no longer R13.2, U3.11, U3.13, U3.15, U3.9
- net IN1: now also R7.2; no longer R8.1
- net IN2: now also R11.2; no longer R10.1
- net IN2_I: now also R9.1; no longer R16.1
- net IN3: now also R17.2; no longer R13.1
- net IN3_I: now also R12.1; no longer R17.1
- net IN4: now also R18.2; no longer R14.1
- net IN4_I: now also R13.1; no longer R18.1
- net VDD: now also U3.10, U3.12, U3.14, U3.16
- net at R11.1: now also R10.1, U3.13; no longer U3.12
- net at U3.3: now also R9.2; no longer R16.2
- net at R12.2: now also U3.5
- net at R7.1: now also R8.1, U3.15; no longer U3.16
- net at U3.7: now also R13.2; no longer R18.2
- new net: R14.1, R17.1, U3.11
- new net: R16.1, R18.1, U3.9
Other:
- note removed: "TODO: make sure those R values make sense"
- moved on the sheet: R15, R8, U3A, U3B, U3C, U3D

Commit message: v3
Parts:
- removed J2: Screw_Terminal_01x04, symbol Connector:Screw_Terminal_01x04
- added J10, J2, J8, J9: Screw_Terminal_01x02, symbol Connector:Screw_Terminal_01x02
Connections:
- net GND: now also J10.2 (Pin_2), J2.2 (Pin_2), J8.2 (Pin_2), J9.2 (Pin_2)
- net IN1_I: now also J2.1 (Pin_1)
- net IN2_I: now also J8.1 (Pin_1)
- net IN3_I: now also J9.1 (Pin_1)
- net IN4_I: now also J10.1 (Pin_1)
Other:
- moved on the sheet: D3, D4, J3, J4, J5, J6, K3, K4, Q7, Q8, R23, R24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

Commit message: ?
Parts:
- J10, J2, J8, J9: footprint (none) -> LIB_TB001-500:CUI_TB001-500-P02BE
- J3, J4, J5, J6: footprint (none) -> LIB_TB010-508:CUI_TB010-508-03BE
- K1, K2, K3, K4: footprint PE014024 -> LIB_PE014024:PE014024
- R10, R11, R12, R13, R14, R15, R16, R17, R18, R19, R20, R21, R22, R23, R24, R25, R26, R7, R8, R9: footprint (none) -> Resistor_SMD:R_0603_1608Metric_Pad0.98x0.95mm_HandSolder
Other:
- company: (none) -> Mateusz Pietrzak, Ruman Mondal, Bassey Bassey
- title: (none) -> Gate controller - inputs and outputs
Changed lines of the file:
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@@
 (kicad_sch (version 20230121) (generator eeschema)
   (paper "A4")
+  (title_block
+    (title "Gate controller - inputs and outputs")
+    (company "Mateusz Pietrzak, Ruman Mondal, Bassey Bassey")
+  )
   (junction (at 154.94 35.56) (diameter 0) (color 0 0 0 0)
   )
@@
       (effects (font (size 1.27 1.27)))
     )
-    (property "Footprint" "" (at 58.42 109.728 90)
+    (property "Footprint" "Resistor_SMD:R_0603_1608Metric_Pad0.98x0.95mm_HandSolder" (at 58.42 109.728 90)
       (effects (font (size 1.27 1.27)) hide)
     )
@@
       (effects (font (size 1.27 1.27)))
     )
-    (property "Footprint" "" (at 142.24 42.418 90)
+    (property "Footprint" "Resistor_SMD:R_0603_1608Metric_Pad0.98x0.95mm_HandSolder" (at 142.24 42.418 90)
       (effects (font (size 1.27 1.27)) hide)
     )
@@
       (effects (font (size 1.27 1.27)) (justify left))
     )
-    (property "Footprint" "" (at 243.84 45.72 0)
+    (property "Footprint" "LIB_TB001-500:CUI_TB001-500-P02BE" (at 243.84 45.72 0)
       (effects (font (size 1.27 1.27)) hide)
     )
@@
       (effects (font (size 1.27 1.27)))
     )
-    (property "Footprint" "" (at 33.02 41.148 90)
+    (property "Footprint" "Resistor_SMD:R_0603_1608Metric_Pad0.98x0.95mm_HandSolder" (at 33.02 41.148 90)
       (effects (font (size 1.27 1.27)) hide)
     )
@@
       (effects (font (size 1.27 1.27)) (justify left))
     )
-    (property "Footprint" "" (at 51.562 146.05 90)
+    (property "Footprint" "Resistor_SMD:R_0603_1608Metric_Pad0.98x0.95mm_HandSolder" (at 51.562 146.05 90)
       (effects (font (size 1.27 1.27)) hide)
     )
@@
       (effects (font (size 1.27 1.27)) (justify left))
     )
-    (property "Footprint" "" (at 243.84 36.83 0)
+    (property "Footprint" "LIB_TB001-500:CUI_TB001-500-P02BE" (at 243.84 36.83 0)
       (effects (font (size 1.27 1.27)) hide)
     )
@@
       (effects (font (size 1.27 1.27)))
     )
-    (property "Footprint" "" (at 142.24 123.698 90)
+    (property "Footprint" "Resistor_SMD:R_0603_1608Metric_Pad0.98x0.95mm_HandSolder" (at 142.24 123.698 90)
       (effects (font (size 1.27 1.27)) hide)
     )
@@
       (effects (font (size 1.27 1.27)))
     )
-    (property "Footprint" "" (at 116.84 77.978 90)
+    (property "Footprint" "Resistor_SMD:R_0603_1608Metric_Pad0.98x0.95mm_HandSolder" (at 116.84 77.978 90)
       (effects (font (size 1.27 1.27)) hide)
     )
@@
       (effects (font (size 1.27 1.27)) (justify left))
     )
-    (property "Footprint" "" (at 243.84 86.36 0)
+    (property "Footprint" "LIB_TB010-508:CUI_TB010-508-03BE" (at 243.84 86.36 0)
       (effects (font (size 1.27 1.27)) hide)
     )
@@
       (effects (font (size 1.27 1.27)) (justify left))
     )
-    (property "Footprint" "" (at 243.84 74.93 0)
+    (property "Footprint" "LIB_TB010-508:CUI_TB010-508-03BE" (at 243.84 74.93 0)
       (effects (font (size 1.27 1.27)) hide)
     )
@@
       (effects (font (size 1.27 1.27)))
     )
-    (property "Footprint" "" (at 142.24 164.338 90)
+    (property "Footprint" "Resistor_SMD:R_0603_1608Metric_Pad0.98x0.95mm_HandSolder" (at 142.24 164.338 90)
       (effects (font (size 1.27 1.27)) hide)
     )
@@
       (effects (font (size 1.27 1.27)) (justify left))
     )
-    (property "Footprint" "" (at 243.84 54.61 0)
+    (property "Footprint" "LIB_TB001-500:CUI_TB001-500-P02BE" (at 243.84 54.61 0)
       (effects (font (size 1.27 1.27)) hide)
     )
@@
       (effects (font (size 1.27 1.27)))
     )
-    (property "Footprint" "" (at 58.42 141.478 90)
+    (property "Footprint" "Resistor_SMD:R_0603_1608Metric_Pad0.98x0.95mm_HandSolder" (at 58.42 141.478 90)
       (effects (font (size 1.27 1.27)) hide)
     )
@@
       (effects (font (size 1.27 1.27)))
     )
-    (property "Footprint" "" (at 142.24 83.058 90)
+    (property "Footprint" "Resistor_SMD:R_0603_1608Metric_Pad0.98x0.95mm_HandSolder" (at 142.24 83.058 90)
       (effects (font (size 1.27 1.27)) hide)
     )
@@
       (effects (font (size 1.27 1.27)))
     )
-    (property "Footprint" "PE014024" (at 195.58 246.05 0)
+    (property "Footprint" "LIB_PE014024:PE014024" (at 195.58 246.05 0)
       (effects (font (size 1.27 1.27)) (justify left top) hide)
     )
@@
       (effects (font (size 1.27 1.27)) (justify left))
     )
-    (property "Footprint" "" (at 51.562 114.3 90)
+    (property "Footprint" "Resistor_SMD:R_0603_1608Metric_Pad0.98x0.95mm_HandSolder" (at 51.562 114.3 90)
       (effects (font (size 1.27 1.27)) hide)
     )
@@
       (effects (font (size 1.27 1.27)))
     )
-    (property "Footprint" "" (at 58.42 46.228 90)
+    (property "Footprint" "Resistor_SMD:R_0603_1608Metric_Pad0.98x0.95mm_HandSolder" (at 58.42 46.228 90)
       (effects (font (size 1.27 1.27)) hide)
     )
@@
       (effects (font (size 1.27 1.27)))
     )
-    (property "Footprint" "PE014024" (at 195.58 205.41 0)
+    (property "Footprint" "LIB_PE014024:PE014024" (at 195.58 205.41 0)
       (effects (font (size 1.27 1.27)) (justify left top) hide)
     )
@@
       (effects (font (size 1.27 1.27)) (justify left))
     )
-    (property "Footprint" "" (at 51.562 82.55 90)
+    (property "Footprint" "Resistor_SMD:R_0603_1608Metric_Pad0.98x0.95mm_HandSolder" (at 51.562 82.55 90)
       (effects (font (size 1.27 1.27)) hide)
     )
@@
       (effects (font (size 1.27 1.27)))
     )
-    (property "Footprint" "PE014024" (at 195.58 164.77 0)
+    (property "Footprint" "LIB_PE014024:PE014024" (at 195.58 164.77 0)
       (effects (font (size 1.27 1.27)) (justify left top) hide)
     )
@@
       (effects (font (size 1.27 1.27)))
     )
-    (property "Footprint" "" (at 116.84 159.258 90)
+    (property "Footprint" "Resistor_SMD:R_0603_1608Metric_Pad0.98x0.95mm_HandSolder" (at 116.84 159.258 90)
       (effects (font (size 1.27 1.27)) hide)
     )
@@
       (effects (font (size 1.27 1.27)))
     )
-    (property "Footprint" "" (at 33.02 136.398 90)
+    (property "Footprint" "Resistor_SMD:R_0603_1608Metric_Pad0.98x0.95mm_HandSolder" (at 33.02 136.398 90)
       (effects (font (size 1.27 1.27)) hide)
     )
@@
       (effects (font (size 1.27 1.27)))
     )
-    (property "Footprint" "" (at 116.84 118.618 90)
+    (property "Footprint" "Resistor_SMD:R_0603_1608Metric_Pad0.98x0.95mm_HandSolder" (at 116.84 118.618 90)
       (effects (font (size 1.27 1.27)) hide)
     )
@@
       (effects (font (size 1.27 1.27)) (justify left))
     )
-    (property "Footprint" "" (at 243.84 27.94 0)
+    (property "Footprint" "LIB_TB001-500:CUI_TB001-500-P02BE" (at 243.84 27.94 0)
       (effects (font (size 1.27 1.27)) hide)
     )
@@
       (effects (font (size 1.27 1.27)) (justify left))
     )
-    (property "Footprint" "" (at 51.562 50.8 90)
+    (property "Footprint" "Resistor_SMD:R_0603_1608Metric_Pad0.98x0.95mm_HandSolder" (at 51.562 50.8 90)
       (effects (font (size 1.27 1.27)) hide)
     )
@@
       (effects (font (size 1.27 1.27)))
     )
-    (property "Footprint" "" (at 33.02 72.898 90)
+    (property "Footprint" "Resistor_SMD:R_0603_1608Metric_Pad0.98x0.95mm_HandSolder" (at 33.02 72.898 90)
       (effects (font (size 1.27 1.27)) hide)
     )
@@
       (effects (font (size 1.27 1.27)))
     )
-    (property "Footprint" "" (at 58.42 77.978 90)
+    (property "Footprint" "Resistor_SMD:R_0603_1608Metric_Pad0.98x0.95mm_HandSolder" (at 58.42 77.978 90)
       (effects (font (size 1.27 1.27)) hide)
     )
@@
       (effects (font (size 1.27 1.27)) (justify left))
     )
-    (property "Footprint" "" (at 243.84 109.22 0)
+    (property "Footprint" "LIB_TB010-508:CUI_TB010-508-03BE" (at 243.84 109.22 0)
       (effects (font (size 1.27 1.27)) hide)
     )
@@
       (effects (font (size 1.27 1.27)))
     )
-    (property "Footprint" "" (at 33.02 104.648 90)
+    (property "Footprint" "Resistor_SMD:R_0603_1608Metric_Pad0.98x0.95mm_HandSolder" (at 33.02 104.648 90)
       (effects (font (size 1.27 1.27)) hide)
     )
@@
       (effects (font (size 1.27 1.27)))
     )
-    (property "Footprint" "PE014024" (at 195.58 124.13 0)
+    (property "Footprint" "LIB_PE014024:PE014024" (at 195.58 124.13 0)
       (effects (font (size 1.27 1.27)) (justify left top) hide)
     )
@@
       (effects (font (size 1.27 1.27)))
     )
-    (property "Footprint" "" (at 116.84 37.338 90)
+    (property "Footprint" "Resistor_SMD:R_0603_1608Metric_Pad0.98x0.95mm_HandSolder" (at 116.84 37.338 90)
       (effects (font (size 1.27 1.27)) hide)
     )
@@
       (effects (font (size 1.27 1.27)) (justify left))
     )
-    (property "Footprint" "" (at 243.84 97.79 0)
-      (effects (font (size 1.27 1.27)) hide)
-    )
+    (property "Footprint" "LIB_TB010-508:CUI_TB010-508-03BE" (at 243.84 97.79 0)
+      (effects (font (size 1.27 1.27)) hide)
+    )
